File: Casquino_Daniel_Shield.kicad_sch (KiCad schematic)
At the start: 12 parts, among them J1 Power, J2 PWM, J3 Analog, J4 PWM, J5 Analog, J6 Communication, J7 Digital

Commit message: buzzer pending
Parts:
- removed Analog_0-7, Analog_8-15, PWM_1x8, Power_1x8: Conn_01x08, Connector_PinHeader_2.54mm:PinHeader_1x08_P2.54mm_Vertical, symbol Connector_Generic:Conn_01x08
- removed PWM_1x10: Conn_01x10, Connector_PinHeader_2.54mm:PinHeader_1x10_P2.54mm_Vertical, symbol Connector_Generic:Conn_01x10
- added BZ1: Buzzer, Buzzer_Beeper:Buzzer_12x9.5RM7.6, symbol Device:Buzzer
- added D1, D2, D3, D4: LED, LED_THT:LED_D5.0mm, symbol Device:LED
- added DHT11: Conn_01x03_Socket, Connector_PinSocket_2.54mm:PinSocket_1x03_P2.54mm_Vertical, symbol Connector:Conn_01x03_Socket
- added I2C, UART1: Conn_01x04, Connector_Molex:Molex_KK-254_AE-6410-04A_1x04_P2.54mm_Vertical, symbol Connector_Generic:Conn_01x04
- added J8: Screw_Terminal_01x02, TerminalBlock_Phoenix:TerminalBlock_Phoenix_MKDS-1,5-2-5.08_1x02_P5.08mm_Horizontal, symbol Connector:Screw_Terminal_01x02
- added LDR: A1050, OptoDevice:R_LDR_D6.4mm_P3.4mm_Vertical, symbol Sensor_Optical:A1050
- added RV1: R_Potentiometer, Potentiometer_THT:Potentiometer_Alps_RK09L_Single_Vertical, symbol Device:R_Potentiometer
- added R_LDR, R_SW1, R_SW2, R_SW_RESET: 10k, Resistor_THT:R_Axial_DIN0207_L6.3mm_D2.5mm_P7.62mm_Horizontal, symbol Device:R
- added R_LED1, R_LED2, R_LED3, R_LED4: 330, Resistor_THT:R_Axial_DIN0207_L6.3mm_D2.5mm_P7.62mm_Horizontal, symbol Device:R
- added SW1, SW2, SW_RESET: SW_Push, Button_Switch_THT:SW_PUSH_6mm, symbol Switch:SW_Push
Connections:
- net *2: now also R_LED1.1
- net *3: now also R_LED2.1
- net *4: now also R_LED3.1
- net *5: now also R_LED4.1
- net +5V: now also DHT11.1 (Pin_1), I2C.3 (Pin_3), LDR.1, RV1.1, SW1.1, SW2.1, SW_RESET.1, UART1.3 (Pin_3)
- net 22: now also DHT11.2 (Pin_2)
- net A0: now also LDR.2, R_LDR.1
- net A1: now also RV1.2
- net GND: now also BZ1.2 (-), D1.1 (K), D2.1 (K), D3.1 (K), D4.1 (K), DHT11.3 (Pin_3), I2C.4 (Pin_4), J8.2 (Pin_2), RV1.3, R_LDR.2, R_SW1.2, R_SW2.2, R_SW_RESET.2, UART1.4 (Pin_4)
- net VCC: now also J8.1 (Pin_1)
- net ~{RESET}: now also R_SW_RESET.1, SW_RESET.2
- new net: D3.2 (A), R_LED3.2
- new net: D4.2 (A), R_LED4.2
- new net: D1.2 (A), R_LED1.2
- new net: D2.2 (A), R_LED2.2
- new net D18: R_SW1.1, SW1.2, UART1.1 (Pin_1)
- new net D19: R_SW2.1, SW2.2, UART1.2 (Pin_2)
- new net D20: I2C.1 (Pin_1)
- new net D21: I2C.2 (Pin_2)
- new net D6: BZ1.1 (+)

Commit message: footprint finished
Parts:
- added D_BUZZER1: 1N4148, Diode_THT:D_DO-35_SOD27_P7.62mm_Horizontal, symbol Diode:1N4148
- added R_BUZZER1: 1k, Resistor_THT:R_Axial_DIN0207_L6.3mm_D2.5mm_P7.62mm_Horizontal, symbol Device:R
- added T_BUZZER1: S8050, Package_TO_SOT_THT:TO-92_Inline, symbol Transistor_BJT:S8050
- RV1: value R_Potentiometer -> POT
- renumbered I2C to I2C1, LDR to LDR1, R_LDR to R_LDR1, R_SW_RESET to R_SW_RESET1, SW_RESET to SW_RESET1
Connections:
- net +5V: now also BZ1.1 (+), D_BUZZER1.1 (K)
- net D6: now also R_BUZZER1.2; no longer BZ1.1 (+)
- net GND: now also T_BUZZER1.1 (E); no longer BZ1.2 (-)
- new net: R_BUZZER1.1, T_BUZZER1.2 (B)
- new net: BZ1.2 (-), D_BUZZER1.2 (A), T_BUZZER1.3 (C)
Other:
- moved on the sheet: BZ1

Commit message: pcb wip
Connections:
- net GND: no longer J1.6 (Pin_6)
Changed lines of the file:
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@@
 	(wire
 		(pts
-			(xy 31.75 44.45) (xy 31.75 46.99)
+			(xy 31.75 40.64) (xy 31.75 46.99)
 		)
 		(stroke

Commit message: todo fix drc
Parts:
- RV1: footprint Potentiometer_THT:Potentiometer_Alps_RK09L_Single_Vertical -> Potentiometer_THT:Potentiometer_Bourns_3386P_Vertical
Connections:
- net D6 is gone; now on net *6: R_BUZZER1.2
- net D18: no longer R_SW1.1, SW1.2
- net D19: no longer R_SW2.1, SW2.2
- net GND: now also J1.6 (Pin_6)
- net RX1/19: now also R_SW2.1, SW2.2
- net TX1/18: now also R_SW1.1, SW1.2

Commit message: fixed schem erc errors
Connections:
- net D18 is gone; now on net TX1/18: UART1.1 (Pin_1)
- net D19 is gone; now on net RX1/19: UART1.2 (Pin_2)
- net D20 is gone; now on net SDA/20: I2C1.1 (Pin_1)
- net D21 is gone; now on net SCL/21: I2C1.2 (Pin_2)

Commit message: fixed template footprints
Parts:
- J1, J3, J4, J5, J6: symbol Connector_Generic:Conn_01x08 -> Connector:Conn_01x08_Socket
- J2: symbol Connector_Generic:Conn_01x10 -> Connector:Conn_01x10_Socket
Connections:
- net GND: no longer J1.6 (Pin_6)
